File: edge_detector.kicad_pcb (KiCad board)
At the start: 4 copper layers, 43 x 20 mm, 57 parts, among them J1 Power, J3 Conn_ARM_SWD_TagConnect_TC2030, Q6 Q_PNP_ECB, SW1 Program, SW2 SW_Push, SW3 SW_Push, U1 HX711, U2 C544396, U3 AMS1117-3.3, U4 MCP73811T-420I-OT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

Commit message: Preparing second order
Parts:
- removed C12: 0.1uF, Capacitor_SMD:C_0402_1005Metric
- removed C13: 10uF, Capacitor_SMD:C_0402_1005Metric
- removed L1: 3.3uH, Inductor_SMD:L_0402_1005Metric
- removed Q6: Q_PNP_ECB, Package_TO_SOT_SMD:SOT-23
- removed R19: 8.2k, Resistor_SMD:R_0402_1005Metric
- removed R22, R23, R24: 1k, Resistor_SMD:R_0402_1005Metric
- removed R4: 10k, Resistor_SMD:R_0402_1005Metric
- added TP1: A-, TestPoint:TestPoint_Pad_1.0x1.0mm, F.Cu at (129.5, 107.0)
- added TP4: E+, TestPoint:TestPoint_Pad_1.0x1.0mm, F.Cu at (129.5, 109.2)
- D1: value LED -> C2286
- J3: moved to B.Cu
- R16, R17: value R -> 10k
- R18: value 20k -> 100k
- SW2: value SW_Push -> Deflate
- SW3: value SW_Push -> Mode
- TP2: value TestPoint -> A+; footprint TestPoint:TestPoint_Pad_1.5x1.5mm -> TestPoint:TestPoint_Pad_1.0x1.0mm
- TP3: value TestPoint -> E-; footprint TestPoint:TestPoint_Pad_1.5x1.5mm -> TestPoint:TestPoint_Pad_1.0x1.0mm
- U1: value HX711 -> AP2112K-3.3; footprint Package_SO:SOP-16_3.9x9.9mm_P1.27mm -> Package_TO_SOT_SMD:SOT-23-5
- U3: value AMS1117-3.3 -> HX710C; footprint Package_TO_SOT_SMD:SOT-89-3 -> Package_SO:SOP-8_3.9x4.9mm_P1.27mm
- U4: value MCP73811T-420I-OT -> C424093
- U5: value ESP32-C3-MINI-1 -> C2838502
- moved U4 31.8 mm to (140.2, 111.3), turned to 180 degrees
- moved R2 28.6 mm to (134.8, 111.8)
- moved U3 27.4 mm to (133.5, 106.8)
- moved D1 23.8 mm to (135.2, 114.2)
- moved R8 20.6 mm to (124.5, 118.2), turned to -90 degrees
- moved R11 18.6 mm to (117.5, 118.2), turned to -90 degrees
- moved R7 18.3 mm to (123.5, 118.2), turned to -90 degrees
- moved C9 17.6 mm to (128.8, 111.8), turned to -90 degrees
- moved R10 17.5 mm to (119.5, 118.2), turned to -90 degrees
- moved R9 17.2 mm to (116.5, 118.3), turned to -90 degrees
- moved C7 17.1 mm to (130.0, 102.8)
- moved C8 17.1 mm to (129.0, 102.8)
- moved R1 16.4 mm to (140.0, 113.8), turned to 0 degrees
- moved R12 15.4 mm to (118.5, 118.2), turned to -90 degrees
- moved TP3 12.9 mm to (127.2, 109.2)
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Connections:
- C14 pad 1: Net-(C13-Pad1) -> GND
- C14 pad 2: GND -> Net-(U3-Vout)
- C15 pad 1: Net-(U1-INA+) -> Net-(U3-IN-)
- C15 pad 2: Net-(U1-INA-) -> Net-(U3-IN+)
- C9 pad 1: +3.3V -> Net-(U3-Vout)
- J3 pad 2: unconnected-(J3-SWDIO-Pad2) -> TXD
- J3 pad 6: unconnected-(J3-SWO-Pad6) -> RXD
- R17 pad 1: +3.3V -> Deflate
- R17 pad 2: Net-(U5-GPIO7) -> GND
- R18 pad 1: Net-(Q6-C) -> +BATT
- R18 pad 2: Net-(U1-VFB) -> Net-(U1-EN)
- R20 pad 1: Net-(U1-INA+) -> Net-(U3-IN-)
- R21 pad 2: Net-(U1-INA-) -> Net-(U3-IN+)
- SW2 pad 1: Net-(U5-GPIO7) -> Deflate
- SW2 pad 2: GND -> +3.3V
- TP2 pad 1: Net-(R20-Pad2) -> Net-(R21-Pad1)
- U1 pad 1: +3.3V -> +BATT
- U1 pad 2: Net-(Q6-B) -> GND
- U1 pad 3: Net-(Q6-C) -> Net-(U1-EN)
- U1 pad 4: Net-(U1-VFB) -> unconnected-(U1-NC-Pad4)
- U1 pad 5: GND -> +3.3V
- U3 pad 1: GND -> Net-(U3-Vout)
- U3 pad 2: +3.3V -> GND
- U3 pad 3: +BATT -> Net-(U3-IN-)
- U5 pad 12: unconnected-(U5-GPIO0/ADC1_CH0/XTAL_32K_P-Pad12) -> HX_DAT
- U5 pad 13: unconnected-(U5-GPIO1/ADC1_CH1/XTAL_32K_N-Pad13) -> HX_SCK
- U5 pad 18: Deflate -> Internal_Vibrator
- U5 pad 19: Internal_Vibrator -> External_Vibrator
- U5 pad 20: External_Vibrator -> SDA
- U5 pad 21: Net-(U5-GPIO7) -> SCL
- U5 pad 22: Net-(U5-GPIO8) -> Deflate
- U5 pad 30: SCL -> RDX
- U5 pad 31: SDA -> TXD
Routing:
- net GND: track 228.8 -> 186.0 mm, vias 2 -> 5
- net +BATT: track 36.1 -> 72.8 mm, vias 1 -> 2
- net Net-(U2B-G): track 2.16 -> 35.5 mm
- net Net-(U2A-G): track 2.16 -> 34.2 mm, vias 0 -> 2
- net HX_DAT: track 0.00 -> 23.6 mm, vias 0 -> 2
- net HX_SCK: track 0.00 -> 21.6 mm, vias 0 -> 2
- net Net-(U4-PROG): track 22.5 -> 1.66 mm, vias 2 -> 0
- net Net-(Q6-C): track 18.8 -> 0.00 mm, vias 3 -> 0
- net External_Vibrator: track 20.5 -> 1.76 mm, vias 2 -> 0
- net Net-(C13-Pad1): track 18.7 -> 0.00 mm, vias 2 -> 0
- net Net-(U5-GPIO7): track 18.6 -> 0.00 mm, vias 2 -> 0
- net Net-(U3-Vout): track 0.00 -> 18.4 mm
- net Net-(Q6-B): track 18.1 -> 0.00 mm
- net TXD: track 0.00 -> 16.2 mm, vias 0 -> 1
- net Net-(U6A-G): track 2.77 -> 18.3 mm, vias 0 -> 2
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Other:
- copper layers 4 -> 2
