File: edge_detector.kicad_sch (KiCad schematic)
At the start: 57 parts, among them J1 Power, J3 Conn_ARM_SWD_TagConnect_TC2030, Q6 C305441, SW1 Program, SW2 SW_Push, SW3 SW_Push, U1 HX711, U2 C544396, U3 C347256, U4 C424093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

Commit message: Preparing second order
Parts:
- removed C12: 0.1uF, Capacitor_SMD:C_0402_1005Metric, symbol Device:C
- removed C13: 10uF, Capacitor_SMD:C_0402_1005Metric, symbol Device:C
- removed L1: 3.3uH, Inductor_SMD:L_0402_1005Metric, symbol Device:L
- removed Q6: C305441, Package_TO_SOT_SMD:SOT-23, symbol Device:Q_PNP_ECB
- removed R19: 8.2k, Resistor_SMD:R_0402_1005Metric, symbol Device:R
- removed R22, R23, R24: 1k, Resistor_SMD:R_0402_1005Metric, symbol Device:R
- removed R4: 10k, Resistor_SMD:R_0402_1005Metric, symbol Device:R
- removed U1: HX711, Package_SO:SOP-16_3.9x9.9mm_P1.27mm, symbol Analog_ADC:HX711
- removed U3: C347256, Package_TO_SOT_SMD:SOT-89-3, symbol Regulator_Linear:AMS1117-3.3
- added TP1: A-, TestPoint:TestPoint_Pad_1.0x1.0mm, symbol Connector:TestPoint
- added TP4: E+, TestPoint:TestPoint_Pad_1.0x1.0mm, symbol Connector:TestPoint
- added U1: AP2112K-3.3, Package_TO_SOT_SMD:SOT-23-5, symbol Regulator_Linear:AP2112K-3.3
- added U3: HX710C, Package_SO:SOP-8_3.9x4.9mm_P1.27mm, symbol Analog_ADC:HX710C
- J1, J3, MPRLS1, SW1: now not fitted
- R18: value 20k -> 100k; LCSC C25765 -> C25741
- SW2: value SW_Push -> Deflate; now not fitted
- SW3: value SW_Push -> Mode; now not fitted
- TP2: value TestPoint -> A+; footprint TestPoint:TestPoint_Pad_1.5x1.5mm -> TestPoint:TestPoint_Pad_1.0x1.0mm; now not fitted
- TP3: value TestPoint -> E-; footprint TestPoint:TestPoint_Pad_1.5x1.5mm -> TestPoint:TestPoint_Pad_1.0x1.0mm; now not fitted
Connections:
- net +3.3V: now also SW2.2, U1.5 (VOUT), U3.7 (VDD); no longer C9.1, R17.1
- net +BATT: now also R18.1, U1.1 (VIN)
- net Deflate: now also R17.1, SW2.1, U5.22 (GPIO8); no longer U5.18 (GPIO4/ADC1_CH4)
- net External_Vibrator: now also U5.19 (GPIO5/ADC2_CH0); no longer U5.20 (GPIO6)
- net GND: now also C14.1, R17.2, U1.2 (GND), U3.2 (AGND); no longer C14.2, SW2.2
- net HX_DAT: now also U5.12 (GPIO0/ADC1_CH0/XTAL_32K_P), U3.6 (DOUT)
- net HX_SCK: now also U5.13 (GPIO1/ADC1_CH1/XTAL_32K_N), U3.5 (PD_SCK)
- net Internal_Vibrator: now also U5.18 (GPIO4/ADC1_CH4); no longer U5.19 (GPIO5/ADC2_CH0)
- net SCL: now also U5.21 (GPIO7); no longer U5.30 (GPIO20/U0RXD)
- net SDA: now also U5.20 (GPIO6); no longer U5.31 (GPIO21/U0TXD)
- net at C15.1, R20.1: now also U3.3 (IN-)
- net at R20.2: now also TP1.1; no longer TP2.1
- net at R21.1: now also TP2.1
- net at C15.2, R21.2: now also U3.4 (IN+)
- net TXD: now reaches J3.2 (SWDIO)
- net TXD: now also U5.31 (GPIO21/U0TXD)
- net RXD: now reaches J3.6 (SWO)
- net at R18.2: now also U1.3 (EN)
- new net: C14.2, C9.1, TP4.1, U3.1 (Vref), U3.8 (Vout)
- new net RDX: U5.30 (GPIO20/U0RXD)
- no-connect marks 11 -> 4
Other:
- moved on the sheet: C10, C11, C14, C15, C3, C5, C9, R17, R20, R21
